Commit message: Added camera_pose to loki.urdf file.

File: loki_description/urdf/loki.urdf (robot description, URDF)
Before this commit: robot loki, 17 links, 16 joints
Links:
- added link camera_pose
Joints:
- added joint base_camera_pose: type fixed, parent base_link, child camera_pose, origin xyz=-0.140 0 0 rpy=0 0 -1.57
