Commit message: update urdf for rev f

File: n_robot_state_publisher/urdf/loki.urdf (robot description, URDF)
Before this commit: robot loki, 18 links, 17 joints
Links:
- removed link camera_pose
- added link raspicam
Joints:
- removed joint base_camera_pose
- added joint base_raspicam: type fixed, parent base_link, child raspicam, origin xyz=-0.15125 0.007 0 rpy=0 0 -1.57
- joint base_sonar_0: origin xyz=-0.117 -0.055 0 rpy=0 0 -1.57 -> xyz=-0.126 -0.0545 -0.015 rpy=3.1416 0 -1.5708
- joint base_sonar_1: origin xyz=0.0540476 -0.0508134 0 rpy=0 0 -1.17 -> xyz=0.04161 -0.044415 0.015 rpy=0 0 -1.1781
- joint base_sonar_10: origin xyz=-0.155890873 0.038890873 0 rpy=0 0 2.35619449 -> xyz=-0.16453732 0.03853732 -0.015 rpy=3.1416 0 2.3562
- joint base_sonar_11: origin xyz=-0.167813374 0.021047589 0 rpy=0 0 2.74889357 -> xyz=-0.176351435 0.020856247 0.015 rpy=0 0 2.7489
- joint base_sonar_12: origin xyz=-0.172 0 0 rpy=0 0 3.14159265 -> xyz=-0.1805 0 -0.015 rpy=3.1416 0 3.1416
- joint base_sonar_13: origin xyz=-0.167813374 -0.021047589 0 rpy=0 0 -2.74889357 -> xyz=-0.176351435 -0.020856247 0.015 rpy=0 0 -2.7489
- joint base_sonar_14: origin xyz=-0.155890873 -0.038890873 0 rpy=0 0 -2.35619449 -> xyz=-0.16453732 -0.03853732 -0.015 rpy=3.1416 0 -2.3562
- joint base_sonar_15: origin xyz=-0.138047589 -0.050813374 0 rpy=0 0 -1.96349541 -> xyz=-0.146856247 -0.050351435 0.015 rpy=0 0 -1.9635
- joint base_sonar_2: origin xyz=0.0718909 -0.0388909 0 rpy=0 0 -0.79 -> xyz=0.06253732 -0.03853732 -0.015 rpy=3.1416 0 -0.7854
- joint base_sonar_3: origin xyz=0.0838134 -0.0210476 0 rpy=0 0 -0.39 -> xyz=0.074351435 -0.020856247 0.015 rpy=0 0 -0.3927
- joint base_sonar_4: origin xyz=0.088 0 0 rpy=0 0 0 -> xyz=0.0785 0 -0.015 rpy=3.1416 0 0
- joint base_sonar_5: origin xyz=0.0838134 0.0210476 0 rpy=0 0 0.39 -> xyz=0.074351435 0.020856247 0.015 rpy=0 0 0.3927
- joint base_sonar_6: origin xyz=0.0718909 0.0388909 0 rpy=0 0 0.79 -> xyz=0.06253732 0.03853732 -0.015 rpy=3.1416 0 0.7854
- joint base_sonar_7: origin xyz=0.0540476 0.0508134 0 rpy=0 0 1.17 -> xyz=0.04131 0.044785 0.015 rpy=0 0 1.1781
- joint base_sonar_8: origin xyz=-0.117 0.055 0 rpy=0 0 1.57 -> xyz=-0.126 0.0545 -0.015 rpy=3.1416 0 1.5708
- joint base_sonar_9: origin xyz=-0.138047589 0.050813374 0 rpy=0 0 1.96349541 -> xyz=-0.146856247 0.050351435 0.015 rpy=0 0 1.9635

Commit message: added sonar mesh

File: n_robot_state_publisher/urdf/loki.urdf (robot description, URDF)
Before this commit: robot loki, 18 links, 17 joints
Links:
- link sonar_0: geometry visual mesh filename=package://ubiquity_launches/n_robot_state_publisher/meshes/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
- link sonar_1: geometry visual mesh filename=package://ubiquity_launches/n_robot_state_publisher/meshes/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
- link sonar_10: geometry visual mesh filename=package://ubiquity_launches/n_robot_state_publisher/meshes/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
- link sonar_11: geometry visual mesh filename=package://ubiquity_launches/n_robot_state_publisher/meshes/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
- link sonar_12: geometry visual mesh filename=package://ubiquity_launches/n_robot_state_publisher/meshes/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
- link sonar_13: geometry visual mesh filename=package://ubiquity_launches/n_robot_state_publisher/meshes/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
- link sonar_14: geometry visual mesh filename=package://ubiquity_launches/n_robot_state_publisher/meshes/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
- link sonar_15: geometry visual mesh filename=package://ubiquity_launches/n_robot_state_publisher/meshes/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
- link sonar_2: geometry visual mesh filename=package://ubiquity_launches/n_robot_state_publisher/meshes/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
- link sonar_3: geometry visual mesh filename=package://ubiquity_launches/n_robot_state_publisher/meshes/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
- link sonar_4: geometry visual mesh filename=package://ubiquity_launches/n_robot_state_publisher/meshes/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
- link sonar_5: geometry visual mesh filename=package://ubiquity_launches/n_robot_state_publisher/meshes/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
- link sonar_6: geometry visual mesh filename=package://ubiquity_launches/n_robot_state_publisher/meshes/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
- link sonar_7: geometry visual mesh filename=package://ubiquity_launches/n_robot_state_publisher/meshes/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
- link sonar_8: geometry visual mesh filename=package://ubiquity_launches/n_robot_state_publisher/meshes/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
- link sonar_9: geometry visual mesh filename=package://ubiquity_launches/n_robot_state_publisher/meshes/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

Commit message: Add angle measurements as comments

File: n_robot_state_publisher/urdf/loki.urdf (robot description, URDF)
Before this commit: robot loki, 18 links, 17 joints
Joints:
- joint base_raspicam: origin xyz=-0.15125 0.007 0 rpy=0 0 -1.57 -> xyz=-0.15125 0.007 0 rpy=0 0 -1.5708

Commit message: Update Loki URDF for Rev F (#2)
* update urdf for rev f

* add comment for sonar top/bottom mounting

* added sonar mesh

* Add angle measurements as comments

File: n_robot_state_publisher/urdf/loki.urdf (robot description, URDF)
Before this commit: robot loki, 18 links, 17 joints
Links:
- removed link camera_pose
- added link raspicam
- link sonar_0: geometry visual mesh filename=package://ubiquity_launches/n_robot_state_publisher/meshes/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
- link sonar_1: geometry visual mesh filename=package://ubiquity_launches/n_robot_state_publisher/meshes/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
- link sonar_10: geometry visual mesh filename=package://ubiquity_launches/n_robot_state_publisher/meshes/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
- link sonar_11: geometry visual mesh filename=package://ubiquity_launches/n_robot_state_publisher/meshes/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
- link sonar_12: geometry visual mesh filename=package://ubiquity_launches/n_robot_state_publisher/meshes/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
- link sonar_13: geometry visual mesh filename=package://ubiquity_launches/n_robot_state_publisher/meshes/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
- link sonar_14: geometry visual mesh filename=package://ubiquity_launches/n_robot_state_publisher/meshes/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
- link sonar_15: geometry visual mesh filename=package://ubiquity_launches/n_robot_state_publisher/meshes/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
- link sonar_2: geometry visual mesh filename=package://ubiquity_launches/n_robot_state_publisher/meshes/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
- link sonar_3: geometry visual mesh filename=package://ubiquity_launches/n_robot_state_publisher/meshes/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
- link sonar_4: geometry visual mesh filename=package://ubiquity_launches/n_robot_state_publisher/meshes/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
- link sonar_5: geometry visual mesh filename=package://ubiquity_launches/n_robot_state_publisher/meshes/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
- link sonar_6: geometry visual mesh filename=package://ubiquity_launches/n_robot_state_publisher/meshes/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
- link sonar_7: geometry visual mesh filename=package://ubiquity_launches/n_robot_state_publisher/meshes/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
- link sonar_8: geometry visual mesh filename=package://ubiquity_launches/n_robot_state_publisher/meshes/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
- link sonar_9: geometry visual mesh filename=package://ubiquity_launches/n_robot_state_publisher/meshes/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
Joints:
- removed joint base_camera_pose
- added joint base_raspicam: type fixed, parent base_link, child raspicam, origin xyz=-0.15125 0.007 0 rpy=0 0 -1.5708
- joint base_sonar_0: origin xyz=-0.117 -0.055 0 rpy=0 0 -1.57 -> xyz=-0.126 -0.0545 -0.015 rpy=3.1416 0 -1.5708
- joint base_sonar_1: origin xyz=0.0540476 -0.0508134 0 rpy=0 0 -1.17 -> xyz=0.04161 -0.044415 0.015 rpy=0 0 -1.1781
- joint base_sonar_10: origin xyz=-0.155890873 0.038890873 0 rpy=0 0 2.35619449 -> xyz=-0.16453732 0.03853732 -0.015 rpy=3.1416 0 2.3562
- joint base_sonar_11: origin xyz=-0.167813374 0.021047589 0 rpy=0 0 2.74889357 -> xyz=-0.176351435 0.020856247 0.015 rpy=0 0 2.7489
- joint base_sonar_12: origin xyz=-0.172 0 0 rpy=0 0 3.14159265 -> xyz=-0.1805 0 -0.015 rpy=3.1416 0 3.1416
- joint base_sonar_13: origin xyz=-0.167813374 -0.021047589 0 rpy=0 0 -2.74889357 -> xyz=-0.176351435 -0.020856247 0.015 rpy=0 0 -2.7489
- joint base_sonar_14: origin xyz=-0.155890873 -0.038890873 0 rpy=0 0 -2.35619449 -> xyz=-0.16453732 -0.03853732 -0.015 rpy=3.1416 0 -2.3562
- joint base_sonar_15: origin xyz=-0.138047589 -0.050813374 0 rpy=0 0 -1.96349541 -> xyz=-0.146856247 -0.050351435 0.015 rpy=0 0 -1.9635
- joint base_sonar_2: origin xyz=0.0718909 -0.0388909 0 rpy=0 0 -0.79 -> xyz=0.06253732 -0.03853732 -0.015 rpy=3.1416 0 -0.7854
- joint base_sonar_3: origin xyz=0.0838134 -0.0210476 0 rpy=0 0 -0.39 -> xyz=0.074351435 -0.020856247 0.015 rpy=0 0 -0.3927
- joint base_sonar_4: origin xyz=0.088 0 0 rpy=0 0 0 -> xyz=0.0785 0 -0.015 rpy=3.1416 0 0
- joint base_sonar_5: origin xyz=0.0838134 0.0210476 0 rpy=0 0 0.39 -> xyz=0.074351435 0.020856247 0.015 rpy=0 0 0.3927
- joint base_sonar_6: origin xyz=0.0718909 0.0388909 0 rpy=0 0 0.79 -> xyz=0.06253732 0.03853732 -0.015 rpy=3.1416 0 0.7854
- joint base_sonar_7: origin xyz=0.0540476 0.0508134 0 rpy=0 0 1.17 -> xyz=0.04131 0.044785 0.015 rpy=0 0 1.1781
- joint base_sonar_8: origin xyz=-0.117 0.055 0 rpy=0 0 1.57 -> xyz=-0.126 0.0545 -0.015 rpy=3.1416 0 1.5708
- joint base_sonar_9: origin xyz=-0.138047589 0.050813374 0 rpy=0 0 1.96349541 -> xyz=-0.146856247 0.050351435 0.015 rpy=0 0 1.9635
